File: eagle/XBee3/Schaltplan1.brd (EAGLE design)
At the start: 102.8 x 84.8 mm, 61 parts, among them IC1 XB3-24Z8CM-J, IC2 317EMP, U1 CONNECTOR_6PIN, X1 22-23-2021, X2 22-23-2031, X3 22-23-2021

Commit message: Board rev0.2
Parts:
- removed TP6, TP7, TP8: TPSQB1,27, testpad:B1,27
- removed U$6: LED_RG_SOT23, ROT_GRÜN_LED_SOT23:SOT23
- added IO11, IO12, IO8: TPSQB1,27, testpad:B1,27
- added LED: LED_RG_SOT23, ROT_GRÜN_LED_SOT23:SOT23
- moved SJ1 43.8 mm to (11.4, 54.6)
- moved X3 43.8 mm to (17.8, 54.6)
- moved X1 43.4 mm to (5.08, 54.6)
- moved SJ5 43.0 mm to (54.6, 11.4), turned to 180 degrees
- moved VCC_EXT 42.6 mm to (24.1, 54.6), turned to 0 degrees
- moved GND1 41.9 mm to (36.8, 54.6), turned to 180 degrees
- moved C1 40.6 mm to (14.0, 30.5)
- moved C2 40.6 mm to (8.89, 30.5)
- moved C3 40.6 mm to (14.0, 26.7)
- moved C4 40.6 mm to (14.0, 22.9)
- moved C5 40.6 mm to (14.0, 19.1)
- moved GND 40.6 mm to (2.54, 49.5)
- moved IC1 40.6 mm to (25.4, 31.8)
- moved R1 40.6 mm to (2.54, 31.8)
- moved R2 40.6 mm to (5.08, 31.8)
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Connections:
- net N$10: now also U1.3; no longer U1.2
- net N$11: now also U1.4; no longer U1.3
- net N$12: now also U1.5; no longer U1.4
- net N$13: now also U1.6; no longer U1.5
- net N$14: now also U1.1; no longer U1.6
- net N$25: now also LED.1; no longer U$6.1
- net N$26: now also LED.2; no longer U$6.2
- net N$3: now also IO12.TP; no longer TP8.TP
- net N$34: now also IO11.TP; no longer TP6.TP
- net N$35: now also IO8.TP; no longer TP7.TP
- net N$43: now also LED.3; no longer U$6.3
- net N$9: now also U1.2; no longer U1.1
Other:
- board size 102.8 x 84.8 mm -> 66 x 58.1 mm
- board text added: "O4"
- board text added: "O5 I1"
- board text added: "O6 I0"
- board text added: "O7 I3"
- board text added: "O9 I2"
- board text added: "Vcc2"

Commit message: Placement grundsätzlich fertig
Parts:
- removed R15, R3, R5, R7, R9: CRCW08050000Z0EA, Resistor_Capacitor:RES_0805
- removed SJ2, SJ3, SJ4, SJ5: (no value), jumper:SJW
- added C10: 100n, Resistor_Capacitor:CAP_0805
- added D1: 5A, Resistor_Capacitor:CAP_0805
- added U$11, U$6: TVS-DIODE, TVS:SOT23-R
- C1, C2, C5: value CC0805KRX7R9BB104 -> 1u
- C3: value CC0805KRX7R9BB104 -> 10u
- C4: value CC0805KRX7R9BB104 -> 85p
- C6, C7, C8, C9: value CC0805KRX7R9BB104 -> 100n
- R1: value CRCW08050000Z0EA -> 150
- R4: value CRCW08050000Z0EA -> 47k
- U$10, U$12, U$7, U$8, U$9: device TVS:SOT23 -> TVS:SOT23-R
- moved R13 29.0 mm to (58.4, 24.1)
- moved C3 28.5 mm to (24.1, 53.3)
- moved U$12 27.1 mm to (14.0, 38.1)
- moved R12 21.7 mm to (55.9, 24.1)
- moved R14 19.1 mm to (44.5, 17.8), turned to 180 degrees
- moved C1 16.7 mm to (16.5, 47.0)
- moved R11 14.8 mm to (53.3, 24.1)
- moved C4 7.62 mm to (14.0, 30.5)
- moved R17 7.18 mm to (12.7, 21.6)
- moved U$10 6.48 mm to (22.9, 17.8)
- moved U$9 6.48 mm to (27.9, 17.8)
- moved U$7 6.48 mm to (38.1, 17.8)
- moved U$8 6.48 mm to (33.0, 17.8)
- moved IO12 2.84 mm to (17.8, 39.4)
- moved IO11 2.84 mm to (17.8, 35.6)
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Connections:
- removed net N$24: R14.1, SJ5.2
- removed net N$36: R11.2, R3.1, U$7.1
- removed net N$37: R12.2, R5.1, U$8.1
- removed net N$38: R13.2, R7.1, U$9.1
- removed net N$39: R14.2, R9.1, U$10.1
- removed net N$40: U$10.3, U$7.3, U$8.3, U$9.3
- removed net N$43: C1.2, C2.2, C3.1, C4.1, C5.2, C6.1, C7.1, C8.1, C9.1, GND.MP, GND1.MP, IC1.1, IC1.10, IC1.12, IC1.21, IC1.32, IC1.34, IC2.1, LED.3, R10.2, R16.2, R4.2, R6.2, R8.2, TP1.TP, U$1.3, U$2.3, U$3.3, U$4.3, U$5.3, UART.1, X1.1, X2.3, X3.1
- removed net N$44: R15.1, R17.2, U$12.1
- removed net N$45: U$12.3
- net N$10: now also R12.1; no longer SJ3.1
- net N$11: now also R13.1; no longer SJ4.1
- net N$12: now also R14.1; no longer SJ5.1
- net N$14: now also D1.1; no longer SJ1.2, U1.1
- net N$15: now also U$11.3
- net N$16: now also C1.2, C10.1, C2.2, C3.1, C4.1, C5.2, C6.1, C7.1, C8.1, C9.1, GND.MP, GND1.MP, IC1.1, IC1.10, IC1.12, IC1.21, IC1.32, IC1.34, IC2.1, LED.3, R10.2, R16.2, R4.2, R6.2, R8.2, TP1.TP, U$1.3, U$2.3, U$3.3, U$4.3, U$5.3, U1.1, X1.1, X2.3, X3.1; no longer IC1.4, UART.2
- net N$17: now also R11.2, U$7.3; no longer R3.2
- net N$18: now also R12.2, U$8.3; no longer R5.2
- net N$19: now also R13.2, U$9.3; no longer R7.2
- net N$2: now also U$10.1, U$11.1, U$12.1, U$6.1, U$7.1, U$8.1, U$9.1, UART.1; no longer R11.1, SJ2.2
- net N$20: now also R14.2, U$10.3; no longer R9.2
- net N$22: now also IC1.4, U$12.3, UART.2; no longer R12.1, SJ3.2
- net N$23: now also D1.2, SJ1.2; no longer R13.1, SJ4.2
- net N$33: now also C10.2, R17.2, U$6.3; no longer R15.2
- net N$41: now also U$11.2, U$6.2
- net N$9: now also R11.1; no longer SJ2.1
Other:
- board size 66 x 58.1 mm -> 66 x 46.7 mm

Commit message: Fertiges Board Vers. Juli 19 (Bestellt)
Parts:
- moved TP1 18.3 mm to (12.7, 26.7)
- moved C2 16.5 mm to (2.54, 45.7), turned to 90 degrees
- moved R2 7.73 mm to (12.7, 33.0), turned to 0 degrees
- moved R1 7.10 mm to (9.53, 33.0), turned to 90 degrees
- moved C10 6.35 mm to (21.6, 21.6), turned to 0 degrees
- moved LED 6.25 mm to (5.08, 32.4), turned to 90 degrees
- moved R11 5.24 mm to (58.4, 22.9)
- moved R13 5.24 mm to (53.3, 22.9)
- moved C9 5.08 mm to (25.4, 21.6), turned to 0 degrees
- moved R16 4.58 mm to (21.6, 24.1), turned to 180 degrees
- moved C8 3.81 mm to (29.2, 21.6), turned to 0 degrees
- moved R10 3.59 mm to (25.4, 24.1), turned to 180 degrees
- moved R4 2.84 mm to (36.8, 24.1), turned to 180 degrees
- moved R8 2.84 mm to (29.2, 24.1), turned to 180 degrees
- moved VCC 2.54 mm to (2.54, 41.9)
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- renumbered IC2 to IC3
Connections:
- removed net N$10: R12.1, U$4.2, U$4.4, U1.3
- removed net N$11: R13.1, U$3.2, U$3.4, U1.4
- removed net N$12: R14.1, U$2.2, U$2.4, U1.5
- removed net N$2: U$10.1, U$11.1, U$12.1, U$6.1, U$7.1, U$8.1, U$9.1, UART.1
- removed net N$41: C1.1, C3.2, C4.2, C5.1, IC1.2, IC3.4, R2.2, U$10.2, U$11.2, U$12.2, U$6.2, U$7.2, U$8.2, U$9.2
- removed net N$9: R11.1, U$5.2, U$5.4, U1.2
- new net GND: C1.2, C10.1, C2.2, C3.1, C4.1, C5.2, C6.1, C7.1, C8.1, C9.1, GND.MP, GND1.MP, IC1.1, IC1.10, IC1.12, IC1.21, IC1.32, IC1.34, IC3.1, LED.3, R10.2, R16.2, R4.2, R6.2, R8.2, TP1.TP, U$1.3, U$10.1, U$11.1, U$12.1, U$2.3, U$3.3, U$4.3, U$5.3, U$6.1, U$7.1, U$8.1, U$9.1, UART.1, X1.1, X2.3, X3.1
- new net N$29: R13.1, U$2.2, U$2.4, U1.5
- new net N$32: R12.1, U$3.2, U$3.4, U1.4
- new net N$36: R11.1, U$4.2, U$4.4, U1.3
- new net VCC: C1.1, C3.2, C4.2, C5.1, IC1.2, IC3.2, IC3.4, R2.2, U$10.2, U$11.2, U$12.2, U$6.2, U$7.2, U$8.2, U$9.2
- net N$13: now also U$5.2, U$5.4, U1.2; no longer U$1.2, U$1.4, U1.6
- net N$14: now also R14.1, U$1.2, U$1.4, U1.6; no longer D1.1, VCC_EXT.MP, X3.2
- net N$16: now also D1.1, VCC_EXT.MP, X3.2; no longer C1.2, C10.1, C2.2, C3.1, C4.1, C5.2, C6.1, C7.1, C8.1, C9.1, GND.MP, GND1.MP, IC1.1, IC1.10, IC1.12, IC1.21, IC1.32, IC1.34, IC3.1, LED.3, R10.2, R16.2, R4.2, R6.2, R8.2, TP1.TP, U$1.3, U$2.3, U$3.3, U$4.3, U$5.3, X1.1, X2.3, X3.1
- net N$17: now also R14.2; no longer R11.2
- net N$18: now also R13.2; no longer R12.2
- net N$19: now also R12.2; no longer R13.2
- net N$20: now also R11.2; no longer R14.2
Routing:
- net GND: track 0.00 -> 126.4 mm, vias 0 -> 38
- net VCC: track 0.00 -> 98.2 mm, vias 0 -> 11
- net N$16: track 0.00 -> 90.6 mm, vias 0 -> 3
- net N$20: track 0.00 -> 74.3 mm, vias 0 -> 2
- net N$19: track 0.00 -> 61.4 mm, vias 0 -> 2
- net N$18: track 0.00 -> 53.7 mm, vias 0 -> 2
- net N$36: track 0.00 -> 40.6 mm
- net N$1: track 0.00 -> 40.3 mm, vias 0 -> 1
- net N$32: track 0.00 -> 37.4 mm
- net N$17: track 0.00 -> 34.3 mm, vias 0 -> 2
- net N$29: track 0.00 -> 31.6 mm
- net N$33: track 0.00 -> 31.0 mm
- net N$8: track 0.00 -> 26.0 mm
- net N$14: track 0.00 -> 26.0 mm
- net N$4: track 0.67 -> 22.5 mm
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- added copper zone on layer 16, net GND
Other:
- board size 66 x 46.7 mm -> 66 x 47.9 mm
- board text added: "GND"
- board text added: "O4 I0"
- board text added: "O5 I3"
- board text added: "O6"
- board text added: "O7 I1"
- board text added: "ext"
- board text removed: "O4"
- board text removed: "O5 I1"
- board text removed: "O6 I0"
- board text removed: "O7 I3"
