File: eagle/XBee3/Schaltplan1.sch (EAGLE design)
At the start: 61 parts, among them IC1 XB3-24Z8CM-J, IC2 317EMP, U1 CONNECTOR_6PIN, X1 22-23-2021, X2 22-23-2031, X3 22-23-2021

Commit message: Board rev0.2
Parts:
- renumbered TP6 to IO11, TP7 to IO8, TP8 to IO12, U$6 to LED
Connections:
- net N$10: now also U1.3; no longer U1.2
- net N$11: now also U1.4; no longer U1.3
- net N$12: now also U1.5; no longer U1.4
- net N$13: now also U1.6; no longer U1.5
- net N$14: now also U1.1; no longer U1.6
- net N$9: now also U1.2; no longer U1.1

Commit message: Placement grundsätzlich fertig
Parts:
- removed R15, R3, R5, R7, R9: CRCW08050000Z0EA, Resistor_Capacitor:CRCW08050000Z0EA
- removed SJ2, SJ3, SJ4, SJ5: (no value), jumper:SJW
- added C10: 100n, Resistor_Capacitor:CC0805KRX7R9BB104
- added D1: 5A, Resistor_Capacitor:CC0805KRX7R9BB104
- added U$11, U$6: TVS-DIODE, TVS:TVS-DIODE
- C1, C2, C5: value CC0805KRX7R9BB104 -> 1u
- C3: value CC0805KRX7R9BB104 -> 10u
- C4: value CC0805KRX7R9BB104 -> 85p
- C6, C7, C8, C9: value CC0805KRX7R9BB104 -> 100n
- R1: value CRCW08050000Z0EA -> 150
- R4: value CRCW08050000Z0EA -> 47k
Connections:
- removed net N$24: R14.1, SJ5.2
- removed net N$36: R11.2, R3.1, U$7.IN
- removed net N$37: R12.2, R5.1, U$8.IN
- removed net N$38: R13.2, R7.1, U$9.IN
- removed net N$39: R14.2, R9.1, U$10.IN
- removed net N$40: U$10.GND, U$7.GND, U$8.GND, U$9.GND
- removed net N$43: C1.2, C2.2, C3.1, C4.1, C5.2, C6.1, C7.1, C8.1, C9.1, GND.MP, GND1.MP, IC1.GND_1, IC1.GND_2, IC1.GND_3, IC1.GND_4, IC1.GND_5, IC1.GND_6, IC2.ADJ, LED.GND, R10.2, R16.2, R4.2, R6.2, R8.2, TP1.TP, U$1.S, U$2.S, U$3.S, U$4.S, U$5.S, UART-1.S, X1-1.S, X2-3.S, X3-1.S
- removed net N$44: R15.1, R17.2, U$12.IN
- removed net N$45: U$12.GND
- net N$10: now also R12.1; no longer SJ3.1
- net N$11: now also R13.1; no longer SJ4.1
- net N$12: now also R14.1; no longer SJ5.1
- net N$14: now also D1.1; no longer SJ1.2, U1.1
- net N$15: now also U$11.IN
- net N$16: now also C1.2, C10.1, C2.2, C3.1, C4.1, C5.2, C6.1, C7.1, C8.1, C9.1, GND.MP, GND1.MP, IC1.GND_1, IC1.GND_2, IC1.GND_3, IC1.GND_4, IC1.GND_5, IC1.GND_6, IC2.ADJ, LED.GND, R10.2, R16.2, R4.2, R6.2, R8.2, TP1.TP, U$1.S, U$2.S, U$3.S, U$4.S, U$5.S, U1.1, X1-1.S, X2-3.S, X3-1.S; no longer IC1.DIN_/_!CONFIG_!/DIO14, UART-2.S
- net N$17: now also R11.2, U$7.IN; no longer R3.2
- net N$18: now also R12.2, U$8.IN; no longer R5.2
- net N$19: now also R13.2, U$9.IN; no longer R7.2
- net N$2: now also U$10.GND, U$11.GND, U$12.GND, U$6.GND, U$7.GND, U$8.GND, U$9.GND, UART-1.S; no longer R11.1, SJ2.2
- net N$20: now also R14.2, U$10.IN; no longer R9.2
- net N$22: now also IC1.DIN_/_!CONFIG_!/DIO14, U$12.IN, UART-2.S; no longer R12.1, SJ3.2
- net N$23: now also D1.2, SJ1.2; no longer R13.1, SJ4.2
- net N$33: now also C10.2, R17.2, U$6.IN; no longer R15.2
- net N$41: now also U$11.VCC, U$6.VCC
- net N$9: now also R11.1; no longer SJ2.1
Other:
- moved on the sheet: C3, C4, GND1, UART-1, UART-2, UART-3

Commit message: Fertiges Board Vers. Juli 19 (Bestellt)
Parts:
- renumbered IC2 to IC3
Connections:
- net N$41 renamed VCC
- removed net N$10: R12.1, U$4.D1, U$4.D2, U1.3
- removed net N$11: R13.1, U$3.D1, U$3.D2, U1.4
- removed net N$12: R14.1, U$2.D1, U$2.D2, U1.5
- removed net N$2: U$10.GND, U$11.GND, U$12.GND, U$6.GND, U$7.GND, U$8.GND, U$9.GND, UART-1.S
- removed net N$9: R11.1, U$5.D1, U$5.D2, U1.2
- new net GND: C1.2, C10.1, C2.2, C3.1, C4.1, C5.2, C6.1, C7.1, C8.1, C9.1, GND.MP, GND1.MP, IC1.GND_1, IC1.GND_2, IC1.GND_3, IC1.GND_4, IC1.GND_5, IC1.GND_6, IC3.ADJ, LED.GND, R10.2, R16.2, R4.2, R6.2, R8.2, TP1.TP, U$1.S, U$10.GND, U$11.GND, U$12.GND, U$2.S, U$3.S, U$4.S, U$5.S, U$6.GND, U$7.GND, U$8.GND, U$9.GND, UART-1.S, X1-1.S, X2-3.S, X3-1.S
- new net N$29: R13.1, U$2.D1, U$2.D2, U1.5
- new net N$32: R12.1, U$3.D1, U$3.D2, U1.4
- new net N$36: R11.1, U$4.D1, U$4.D2, U1.3
- net N$13: now also U$5.D1, U$5.D2, U1.2; no longer U$1.D1, U$1.D2, U1.6
- net N$14: now also R14.1, U$1.D1, U$1.D2, U1.6; no longer D1.1, VCC_EXT.MP, X3-2.S
- net N$16: now also D1.1, VCC_EXT.MP, X3-2.S; no longer C1.2, C10.1, C2.2, C3.1, C4.1, C5.2, C6.1, C7.1, C8.1, C9.1, GND.MP, GND1.MP, IC1.GND_1, IC1.GND_2, IC1.GND_3, IC1.GND_4, IC1.GND_5, IC1.GND_6, IC3.ADJ, LED.GND, R10.2, R16.2, R4.2, R6.2, R8.2, TP1.TP, U$1.S, U$2.S, U$3.S, U$4.S, U$5.S, X1-1.S, X2-3.S, X3-1.S
- net N$17: now also R14.2; no longer R11.2
- net N$18: now also R13.2; no longer R12.2
- net N$19: now also R12.2; no longer R13.2
- net N$20: now also R11.2; no longer R14.2
Other:
- moved on the sheet: R10, R11, R12, R13, R14, R17
